File: PX4FMUv2.3.brd (EAGLE design)
At the start: 70 x 40.5 mm, 252 parts, among them J201 DF13C-6P-1.25V, J202 DF13C-6P-1.25V, J203 DF13C-6P-1.25V, J204 DF13C-6P-1.25V, J301 47346-0001, J302 DF13C-4P-1.25V, J401 DF13C-4P-1.25V, J402 DF13C-3P-1.25V, J403 DF13C-7P-1.25V, J404 DF13C-5P-1.25V, J405 DF13C-4P-1.25V, J601 DF13C-6P-1.25V, J701 DF13C-2P-1.25V, J702 DF13C-3P-1.25V, J801 JST-ZH-3, M3_MOUNT1101 MOUNT-HOLE3.1MM, M3_MOUNT1102 MOUNT-HOLE3.1MM, M3_MOUNT1103 MOUNT-HOLE3.1MM, M3_MOUNT1104 MOUNT-HOLE3.1MM, U101 STM32F4X7VX, U102 FM25V01, U201 TXS0108QFN20, U202 TXS0108QFN20, U301 2908-05WB-MG, U401 MAX3051, U501 L3GD20, U502 L3GD20H, U503 MS5611-01BA, U701 TCA62724FMG, U702 LT3469, U703 LRTB GFTG-T7AW-1+V7A7-29+R5T9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, U801 STM32F10XCXT6, U901 TXS0108QFN20, U902 TXS0108QFN20, U903 74LVC2G240, X101 3.2x2.5 mm / 24 MHz / 15 ppm, X801 3.2x2.5 mm / 24 MHz / 15 ppm

Commit message: Updates to reflect questions asked on mailing list https://groups.google.com/forum/#!topicsearchin/px4users/mosfet%7Csort:date/px4users/fcfwdMKPhbI
Parts:
- B601: value MS621FE -> DO NOT PLACE
- U$3, U$4, U$5: value MOSFET-DUAL-PCHANNEL-CHIPFET -> NTHD4102P
Changed lines of the file:
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@@
 <?xml version="1.0" encoding="utf-8"?>
 <!DOCTYPE eagle SYSTEM "eagle.dtd">
-<eagle version="6.5.0">
+<eagle version="6.4">
 <drawing>
 <settings>
@@
 <attribute name="PARTNO" value="DF13C-4P-1.25V(20)" x="42.672" y="34.7472" size="1.778" layer="28" rot="MR270" display="off"/>
 </element>
-<element name="B601" library="pixhawk2" package="MS621FE" value="MS621FE" x="18.8928" y="28.2704">
+<element name="B601" library="pixhawk2" package="MS621FE" value="DO NOT PLACE" x="18.8928" y="28.2704">
 <attribute name="MFGPN" value="MS621FE" x="18.8928" y="28.2704" size="1.778" layer="27" display="off"/>
 <attribute name="DATASHEET" value="http://speed.sii.co.jp/data/file_PRODUCT_MASTER_50112_TITLE_IMAGESP.pdf" x="18.8928" y="28.2704" size="1.778" layer="27" display="off"/>
@@
 <attribute name="PARTNO" value="*" x="61.8744" y="33.3248" size="1.778" layer="27" display="off"/>
 </element>
-<element name="U$3" library="pixhawk2" package="1206-8" value="MOSFET-DUAL-PCHANNEL-CHIPFET" x="66.4464" y="36.6776" rot="R270">
+<element name="U$3" library="pixhawk2" package="1206-8" value="NTHD4102P" x="66.4464" y="36.6776" rot="R270">
 <attribute name="PARTNO" value="*" x="66.4464" y="36.6776" size="1.778" layer="27" rot="R270" display="off"/>
 </element>
-<element name="U$4" library="pixhawk2" package="1206-8" value="MOSFET-DUAL-PCHANNEL-CHIPFET" x="66.4464" y="32.8168" rot="R270">
+<element name="U$4" library="pixhawk2" package="1206-8" value="NTHD4102P" x="66.4464" y="32.8168" rot="R270">
 <attribute name="PARTNO" value="*" x="66.4464" y="32.8168" size="1.778" layer="27" rot="R270" display="off"/>
 </element>
-<element name="U$5" library="pixhawk2" package="1206-8" value="MOSFET-DUAL-PCHANNEL-CHIPFET" x="66.4464" y="29.0576" rot="R270">
+<element name="U$5" library="pixhawk2" package="1206-8" value="NTHD4102P" x="66.4464" y="29.0576" rot="R270">
 <attribute name="PARTNO" value="*" x="66.4464" y="29.0576" size="1.778" layer="27" rot="R270" display="off"/>
 </element>
