File: PX4FMUv2.4.5.brd (EAGLE design)
At the start: 70 x 40.5 mm, 292 parts, among them J201 DF13C-6P-1.25V, J202 DF13C-6P-1.25V, J203 DF13C-6P-1.25V, J204 DF13C-6P-1.25V, J301 47346-0001, J302 DF13C-4P-1.25V, J401 DF13C-4P-1.25V, J402 DF13C-3P-1.25V, J403 DF13C-7P-1.25V, J404 DF13C-5P-1.25V, J405 DF13C-4P-1.25V, J601 DF13C-6P-1.25V, J701 DF13C-2P-1.25V, J702 DF13C-3P-1.25V, J801 JST-ZH-3, M3_MOUNT1101 MOUNT-HOLE3.1MM, M3_MOUNT1102 MOUNT-HOLE3.1MM, M3_MOUNT1103 MOUNT-HOLE3.1MM, M3_MOUNT1104 MOUNT-HOLE3.1MM, Q601 MMBT3906LT1SMD, U1001 BQ24313, U1002 MIC5332, U101 STM32F4X7VX, U102 FM25V01, U1101 LTC4417, U1102 NTHD4102PT1G, U1103 NTHD4102PT1G, U1104 NTHD4102PT1G, U201 TXS0108QFN20, U202 TXS0108QFN20, U301 2908-05WB-MG, U302 NUF2042XV6, U401 MAX3051, U501 L3GD20, U502 L3GD20H, U504 LSM303D, U505 MPU-6000, U506 MS5611-01BA, U601 BQ24315, U602 BQ24315, U603 MIC5332, U701 TCA62724FMG, U702 LT3469, U703 LRTB GFTG-T7AW-1+V7A7-29+R5T9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, U801 STM32F10XCXT6, U901 TXS0108QFN20, U902 TXS0108QFN20, U903 74LVC2G240, X101 3.2x2.5 mm / 24 MHz / 15 ppm, X503 0512811094, X801 3.2x2.5 mm / 24 MHz / 15 ppm

Commit message: FMU v2.4.5 sch mistake fix - C1110 to 10p
Parts:
- C1110: value 1000p/25V -> 10p/25V
Changed lines of the file:
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@@
 <?xml version="1.0" encoding="utf-8"?>
 <!DOCTYPE eagle SYSTEM "eagle.dtd">
-<eagle version="6.5.0">
+<eagle version="7.1.0">
 <drawing>
 <settings>
@@
 <pass name="Default">
 <param name="RoutingGrid" value="50mil"/>
+<param name="AutoGrid" value="1"/>
+<param name="Efforts" value="0"/>
+<param name="TopRouterVariant" value="1"/>
 <param name="tpViaShape" value="round"/>
 <param name="PrefDir.1" value="|"/>
@@
 <attribute name="PARTNO" value="C0402C100J3GACTU" x="58.3184" y="33.2232" size="1.778" layer="27" rot="R270" display="off"/>
 </element>
-<element name="C1110" library="pixhawk2" package="0402-CAP" value="1000p/25V" x="58.3184" y="30.5816" rot="R270">
-<attribute name="PARTNO" value="GRM1555C1E102JA01D" x="58.3184" y="30.5816" size="1.778" layer="27" rot="R270" display="off"/>
+<element name="C1110" library="pixhawk2" package="0402-CAP" value="10p/25V" x="58.3184" y="30.5816" rot="R270">
+<attribute name="PARTNO" value="C0402C100J3GACTU" x="58.3184" y="30.5816" size="1.778" layer="27" rot="R270" display="off"/>
 </element>
 <element name="C615" library="pixhawk2" package="0402-CAP" value="0u1" x="53.6448" y="13.8176" rot="R180">
