File: sapog_reference_hardware/sapog_reference_hardware.sch (EAGLE design)
At the start: 101 parts, among them CON1 SM06B-SRSS-TB, CON2 CON-4P-RA-JST_GH, CON3 CON-4P-RA-JST_GH, CON4 CON-4P-RA-JST_GH, CON5 CON-4P-RA-JST_GH, IC1 STM32F105, IC2 CAT24C02, IC3 SN65HVD232D, IC4 SN65HVD232D, IC5 LM75BD-TSSOP8, IC6 FAN7888, IC7 ZXCT1051, IC8 3.3V, Q1 BSC019N04NS-DFN5X6, Q2 BSC019N04NS-DFN5X6, Q3 BSC019N04NS-DFN5X6, Q4 BSC019N04NS-DFN5X6, Q5 BSC019N04NS-DFN5X6, Q6 BSC019N04NS-DFN5X6, X1 24MHz

Commit message: Fixed the BOM entry of the power decoupling capacitor. 25 V tantalum capacitors degrade quickly, the new recommendation is to use 35 V rated capacitors. For more info, see https://forum.zubax.com/t/configuring-orel-for-particular-motor/80/23?u=pavel-kirienko
Parts:
- C35: ALTERNATE#1 718-1886-1-ND -> (none); ALTERNATE#2 399-5221-1-ND -> (none)
Changed lines of the file:
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@@
 <part name="R7" library="R_digikey" deviceset="3K9" device="-0402" technology="-1%" value="3K9"/>
 <part name="C35" library="sapog_reference_hardware" deviceset="C-TANT" device="-3024" value="100µF">
-<attribute name="ALTERNATE#1" value="718-1886-1-ND"/>
-<attribute name="ALTERNATE#2" value="399-5221-1-ND"/>
 </part>
 <part name="GND44" library="sapog_reference_hardware" deviceset="GND" device=""/>
